Commit message: extended front bonet

File: model/vehicle.xacro (robot description, xacro)
@@ -50,4 +50,5 @@
   <xacro:property name="body_inertia_z" value="${1.0/12.0 * body_mass * (body_length*body_length + body_width*body_width)}"/>
   <xacro:property name="wheel_separation" value="${body_width + wheel_width}"/>
+  <xacro:property name="wheel_offset_front" value="${body_length/2 - (wheel_radius * 2)}"/>
   <xacro:property name="wheel_offset" value="${body_length/2 - wheel_radius}"/>
   <xacro:property name="wheel_mass" value="${wheel_density * PI * wheel_radius * wheel_radius * wheel_width}"/>
@@ -267,5 +268,5 @@
   <!-- Front Left Steering Joint -->
   <joint name="front_left_steering_joint" type="revolute">
-    <origin xyz="${wheel_offset} ${wheel_separation/2} -${wheel_radius/2}" rpy="0 0 0"/>
+    <origin xyz="${wheel_offset_front} ${wheel_separation/2} -${wheel_radius/2}" rpy="0 0 0"/>
     <parent link="body_link"/>
     <child link="front_left_steering_link"/>
@@ -285,5 +286,5 @@
   <!-- Front Right Steering Joint -->
   <joint name="front_right_steering_joint" type="revolute">
-    <origin xyz="${wheel_offset} ${-wheel_separation/2} -${wheel_radius/2}" rpy="0 0 0"/>
+    <origin xyz="${wheel_offset_front} ${-wheel_separation/2} -${wheel_radius/2}" rpy="0 0 0"/>
     <parent link="body_link"/>
     <child link="front_right_steering_link"/>
